Commit message: changes to node

File: panda_cnr_description/urdf/panda_cnr.xacro (robot description, xacro)
@@ -1,10 +1,10 @@
 <?xml version="1.0"?>
-<robot xmlns:xacro="http://ros.org/wiki/xacro" name="cell" >
+<robot xmlns:xacro="http://ros.org/wiki/xacro" name="panda_cnr" >
 <xacro:include filename="$(find franka_description)/robots/panda_arm_hand.urdf.xacro" />
 <link name="world"/>
-  <joint name="world2panda" type="fixed">
-    <parent link="world"/>
-    <child link="panda_link0"/>
-    <origin xyz="0 0.5 0"/>
-  </joint>
+<joint name="world2panda" type="fixed">
+  <parent link="world"/>
+  <child link="panda_link0"/>
+  <origin xyz="0 0 0"/>
+</joint>
 </robot>
